Commit message: simulation with Gazebo

File: src/edabot_description/urdf/edabot.ros2_control.xacro (robot description, xacro)
@@ -2,8 +2,17 @@
 <robot xmlns:xacro="http://www.ros.org/wiki/xacro" name="edabot">
     <ros2_control type="system" name="RobotSystem">
-        <hardware>
-            <plugin>edabot_firmware/EdabotInterface</plugin>
-            <param name="port">/dev/ttyACM0</param>
-        </hardware>
+        <!-- gazebo -->
+        <xacro:if value="$(arg is_sim)">
+            <hardware>
+                <plugin>gazebo_ros2_control/GazeboSystem</plugin>
+            </hardware>
+        </xacro:if>
+        <!-- robot hardware -->
+        <xacro:unless value="$(arg is_sim)">
+            <hardware>
+                <plugin>amar_firmware/AmarInterface</plugin>
+                <param name="port">/dev/ttyACM0</param>
+            </hardware>
+        </xacro:unless>
         <!-- ros2_control common interfaces -->
         <joint name="base_to_right_wheel_joint">

File: src/edabot_description/urdf/edabot.urdf.xacro (robot description, xacro)
@@ -1,6 +1,9 @@
 <?xml version="1.0"?>
 <robot xmlns:xacro="http://www.ros.org/wiki/xacro" name="edabot">
+    <xacro:arg name="is_sim" default="true"/>
     <!-- include ros2_control -->
     <xacro:include filename="$(find edabot_description)/urdf/edabot.ros2_control.xacro"/>
+    <!-- include ros2_control and gazebo -->
+    <xacro:include filename="$(find edabot_description)/urdf/edabot.gazebo.xacro"/>
     <!-- some material common properties (color) -->
     <material name="white">
@@ -115,5 +118,5 @@
         <child link="left_wheel_link"/>
         <origin xyz="0 ${(base_width/2)} ${-((base_height/2) - wheel_radius) - 0.0375}" rpy="-${pi/2} 0 0"/>
-        <axis xyz="0 0 -1"/>
+        <axis xyz="0 0 1"/>
     </joint>
     <!-- caster wheel front link and joint -->
