Commit message: Mengganti src dengan kode 2BumperBot dari lokal

File: src/bumperbot_description/urdf/bumperbot.urdf.xacro (robot description, xacro)
@@ -15,5 +15,5 @@
   <xacro:property name="base_mass" value="20.0"/>
   <xacro:property name="wheel_radius" value="0.075"/>
-  <xacro:property name="wheel_thickness" value="0.075"/>
+  <xacro:property name="wheel_thickness" value="0.04"/>
   <xacro:property name="wheel_mass" value="0.23"/>
   <xacro:property name="caster_wheel_radius" value="0.05"/>

File: src/bumperbot_description/urdf/bumperbot_ros2_control.xacro (robot description, xacro)
@@ -21,5 +21,5 @@
             <hardware>
                 <plugin>bumperbot_firmware/BumperbotInterface</plugin>
-                <param name="port">/dev/arduino</param>
+                <param name="port">/dev/ttyUSB0</param>
             </hardware>
         </xacro:unless>

Commit message: update

File: src/bumperbot_description/urdf/bumperbot.urdf.xacro (robot description, xacro)
@@ -233,5 +233,5 @@
   </joint>
   -->
-  <!-- <link name="imu_link">
+ <link name="imu_link">
     <inertial>
       <origin xyz="-0.00552433659106688 0.000168210391520346 0.000514000497342681" rpy="0 0 0" />
@@ -257,8 +257,8 @@
   <joint name="imu_joint" type="fixed">
     <origin xyz="0 0 0.0698986241758014" rpy="0 0 0" />
-    <parent link="base_link" />
+    <parent link="base_footprint" />
     <child link="imu_link" />
     <axis xyz="0 0 0" />
-  </joint> -->
+  </joint>
   <link name="laser_link">
     <inertial>
